Commit message: minor bugs fixed

File: universal_robot/ur_description/urdf/b.urdf (robot description, URDF)
Before this commit: robot ur10.gripper, 22 links, 21 joints
Joints:
- joint world_joint: origin xyz=0.0 0.0 0.4 rpy=0.0 0.0 0.0 -> xyz=0.0 0.0 0.8 rpy=0.0 0.0 0.0

File: universal_robot/ur_description/urdf/c.urdf (robot description, URDF)
Before this commit: robot ur10.gripper, 22 links, 21 joints
Joints:
- joint world_joint: origin xyz=0.0 0.0 0.4 rpy=0.0 0.0 0.0 -> xyz=0.0 0.0 0.8 rpy=0.0 0.0 0.0

File: universal_robot/ur_description/urdf/ur10_gripper.urdf.xacro (robot description, xacro)
@@ -15,5 +15,6 @@
 		 wrist_1_lower_limit="${-pi}" wrist_1_upper_limit="${pi}"
 		 wrist_2_lower_limit="${-pi}" wrist_2_upper_limit="${pi}"
-		 wrist_3_lower_limit="${-pi}" wrist_3_upper_limit="${pi}" />
+		 wrist_3_lower_limit="${-pi}" wrist_3_upper_limit="${pi}"
+/>
   <!-- gripper -->
   <xacro:pr2_gripper_v0 reflect="-1.0" side="r" parent="ee_link"
@@ -34,5 +35,5 @@
     <parent link="world" />
     <child link = "base_link" />
-    <origin xyz="0.0 0.0 0.4" rpy="0.0 0.0 0.0" />
+    <origin xyz="0.0 0.0 0.8" rpy="0.0 0.0 0.0" />
   </joint>
 </robot>
