Commit message: controller fixed

File: universal_robot/ur_description/urdf/d.urdf (robot description, URDF)
Before this commit: robot ur10.gripper, 22 links, 21 joints
Joints:
- joint ee_fixed_joint: origin xyz=0.0 0.0622 0.0 rpy=0.0 0.0 1.57079632679 -> xyz=0.0 0.0922 0.0 rpy=0.0 0.0 1.57079632679
